File: PCB/OSHE-Reader-Buttons.kicad_sch (KiCad schematic)
At the start: 10 parts, among them SW1 SW_Push, SW2 SW_Push, SW3 SW_Push, SW4 SW_Push, SW5 SW_Push

Commit message: small
Connections:
- net RightButton is gone; now on net DownScreenbutton: R17.1, SW2.2
- net UpButton is gone; now on net UpScreenbutton: R14.1, SW3.2
- removed net 3V3: SW1.1, SW2.1, SW3.1, SW4.1, SW5.1
- net DownButton renamed DownScreenbutton
- net LeftButton renamed UpScreenbutton
- new net buttonDownLeft: SW4.1
- new net buttonDownRight: SW2.1
- new net buttonUpLeft: SW3.1
- new net buttonUpRight: SW1.1
- new net centerButton: SW5.1
Changed lines of the file:
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@@
 	)
 	(hierarchical_label "GND"
-		(shape input)
+		(shape output)
 		(at 140.97 64.77 270)
 		(effects
@@
 	)
 	(hierarchical_label "GND"
-		(shape input)
+		(shape output)
 		(at 66.04 93.98 270)
 		(effects
@@
 		)
 	)
-	(hierarchical_label "3V3"
+	(hierarchical_label "buttonUpRight"
 		(shape input)
 		(at 116.84 38.1 180)
@@
 		)
 	)
-	(hierarchical_label "DownButton"
+	(hierarchical_label "DownScreenbutton"
 		(shape output)
 		(at 69.85 73.66 0)
@@
 		)
 	)
-	(hierarchical_label "LeftButton"
+	(hierarchical_label "UpScreenbutton"
 		(shape output)
 		(at 153.67 49.53 0)
@@
 		)
 	)
-	(hierarchical_label "3V3"
+	(hierarchical_label "buttonUpLeft"
 		(shape input)
 		(at 40.64 36.83 180)
@@
 		)
 	)
-	(hierarchical_label "UpButton"
+	(hierarchical_label "UpScreenbutton"
 		(shape output)
 		(at 73.66 46.99 0)
@@
 		)
 	)
-	(hierarchical_label "3V3"
+	(hierarchical_label "buttonDownRight"
 		(shape input)
 		(at 116.84 63.5 180)
@@
 		)
 	)
-	(hierarchical_label "3V3"
+	(hierarchical_label "buttonDownLeft"
 		(shape input)
 		(at 40.64 62.23 180)
@@
 	)
 	(hierarchical_label "GND"
-		(shape input)
+		(shape output)
 		(at 113.03 113.03 270)
 		(effects
@@
 		)
 	)
-	(hierarchical_label "RightButton"
+	(hierarchical_label "DownScreenbutton"
 		(shape output)
 		(at 144.78 73.66 0)
@@
 	)
 	(hierarchical_label "GND"
-		(shape input)
+		(shape output)
 		(at 66.04 58.42 270)
 		(effects
@@
 		)
 	)
-	(hierarchical_label "3V3"
+	(hierarchical_label "centerButton"
 		(shape input)
 		(at 93.98 81.28 180)
@@
 	)
 	(hierarchical_label "GND"
-		(shape input)
+		(shape output)
 		(at 139.7 93.98 270)
 		(effects
