File: PCB/OSHE-Reader-Display-Connector.kicad_sch (KiCad schematic)
At the start: 18 parts, among them J3 Conn_01x24_MountingPin, Q2 Si1308EDL

Commit message: small
Parts:
- renumbered C14 to C13, C15 to C14, C18 to C17, C19 to C18, C20 to C19, C21 to C20, C22 to C21, C23 to C22, C17 to C?, C16 to C?, D1 to D?, J3 to J?, L2 to L?, Q2 to Q?, R19 to R?
Connections:
- net VCOM: now reaches C22.1, J?.24 (VCOM)
- net GND renamed BS
- net RESET renamed RES
Other:
- moved on the sheet: C13, C17, C18, C19, C20, C21, C22, C?, J?, L?
