File: PCB/OSHE-Reader-Battery.kicad_sch (KiCad schematic)
At the start: 11 parts, among them Q1 PNP, U1 BQ2057CSNTR, U2 IRF7326D2TRPBF

Commit message: Update OSHE-Reader-Battery.kicad_sch
Parts:
- added TH2: 10K, symbol Device:Thermistor_NTC
Connections:
- net GND: now also TH2.2
- net TS: now also TH2.1
Other:
- moved on the sheet: R3, R4
Changed lines of the file:
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@@
 	)
 	(junction
-		(at 26.67 99.06)
+		(at 39.37 99.06)
 		(diameter 0)
 		(color 0 0 0 0)
@@
 	(wire
 		(pts
-			(xy 26.67 87.63) (xy 26.67 85.09)
+			(xy 25.4 109.22) (xy 25.4 106.68)
+		)
+		(stroke
+			(width 0)
+			(type default)
+		)
+	)
+	(wire
+		(pts
+			(xy 39.37 87.63) (xy 39.37 85.09)
 		)
 		(stroke
@@
 	(wire
 		(pts
-			(xy 26.67 99.06) (xy 29.21 99.06)
-		)
-		(stroke
-			(width 0)
-			(type default)
-		)
-	)
-	(wire
-		(pts
 			(xy 71.12 110.49) (xy 71.12 113.03)
 		)
@@
 	(wire
 		(pts
+			(xy 39.37 99.06) (xy 44.45 99.06)
+		)
+		(stroke
+			(width 0)
+			(type default)
+		)
+	)
+	(wire
+		(pts
 			(xy 137.16 97.79) (xy 137.16 100.33)
 		)
@@
 	(wire
 		(pts
-			(xy 26.67 113.03) (xy 26.67 110.49)
+			(xy 39.37 113.03) (xy 39.37 110.49)
 		)
 		(stroke
@@
 	(wire
 		(pts
-			(xy 26.67 102.87) (xy 26.67 99.06)
+			(xy 39.37 102.87) (xy 39.37 99.06)
 		)
 		(stroke
@@
 	(wire
 		(pts
-			(xy 26.67 99.06) (xy 26.67 95.25)
+			(xy 39.37 99.06) (xy 39.37 95.25)
+		)
+		(stroke
+			(width 0)
+			(type default)
+		)
+	)
+	(wire
+		(pts
+			(xy 25.4 99.06) (xy 39.37 99.06)
 		)
 		(stroke
@@
 	(hierarchical_label "GND"
 		(shape input)
-		(at 26.67 113.03 270)
+		(at 39.37 113.03 270)
 		(effects
 			(font
@@
 	(hierarchical_label "TS"
 		(shape passive)
-		(at 29.21 99.06 0)
+		(at 44.45 99.06 0)
 		(effects
 			(font
@@
 	(hierarchical_label "VBUS"
 		(shape input)
-		(at 26.67 85.09 90)
+		(at 39.37 85.09 90)
 		(effects
 			(font
@@
 		(shape passive)
 		(at 36.83 60.96 180)
+		(effects
+			(font
+				(size 1.27 1.27)
+			)
+			(justify right)
+		)
+	)
+	(hierarchical_label "GND"
+		(shape input)
+		(at 25.4 109.22 270)
 		(effects
 			(font
@@
 	(symbol
 		(lib_id "Device:R")
-		(at 26.67 106.68 0)
+		(at 39.37 106.68 0)
 		(unit 1)
 		(exclude_from_sim no)
@@
 		(fields_autoplaced yes)
 		(property "Reference" "R4"
-			(at 29.21 105.4099 0)
+			(at 41.91 105.4099 0)
 			(effects
 				(font
@@
 		)
 		(property "Value" "R_{T1}/100K"
-			(at 29.21 107.9499 0)
+			(at 41.91 107.9499 0)
 			(effects
 				(font
@@
 		)
 		(property "Footprint" ""
-			(at 24.892 106.68 90)
+			(at 37.592 106.68 90)
 			(effects
 				(font
@@
 		)
 		(property "Datasheet" "~"
-			(at 26.67 106.68 0)
+			(at 39.37 106.68 0)
 			(effects
 				(font
@@
 		)
 		(property "Description" "Resistor"
-			(at 26.67 106.68 0)
+			(at 39.37 106.68 0)
 			(effects
 				(font
@@
 				(path "/3f072c92-e35a-4654-839b-728bd3dc3a46/9b683008-b3f5-4049-bcf9-7e8cdd298ddd"
 					(reference "R4")
+					(unit 1)
+				)
+			)
+		)
+	)
+	(symbol
+		(lib_id "Device:Thermistor_NTC")
+		(at 25.4 102.87 0)
+		(unit 1)
+		(exclude_from_sim no)
+		(in_bom yes)
+		(on_board yes)
+		(dnp no)
+		(fields_autoplaced yes)
+		(property "Reference" "TH2"
+			(at 27.94 101.9174 0)
+			(effects
+				(font
+					(size 1.27 1.27)
+				)
+				(justify left)
+			)
+		)
+		(property "Value" "10K"
+			(at 27.94 104.4574 0)
+			(effects
+				(font
+					(size 1.27 1.27)
+				)
+				(justify left)
+			)
+		)
+		(property "Footprint" ""
+			(at 25.4 101.6 0)
+			(effects
+				(font
+					(size 1.27 1.27)
+				)
+				(hide yes)
+			)
+		)
+		(property "Datasheet" "~"
+			(at 25.4 101.6 0)
+			(effects
+				(font
+					(size 1.27 1.27)
+				)
+				(hide yes)
+			)
+		)
+		(property "Description" "Temperature dependent resistor, negative temperature coefficient"
+			(at 25.4 102.87 0)
+			(effects
+				(font
+					(size 1.27 1.27)
+				)
+				(hide yes)
+			)
+		)
+		(pin "1"
+		)
+		(pin "2"
+		)
+		(instances
+			(project ""
+				(path "/3f072c92-e35a-4654-839b-728bd3dc3a46/9b683008-b3f5-4049-bcf9-7e8cdd298ddd"
+					(reference "TH2")
 					(unit 1)
 				)
@@
 	(symbol
 		(lib_id "Device:R")
-		(at 26.67 91.44 0)
+		(at 39.37 91.44 0)
 		(unit 1)
 		(exclude_from_sim no)
@@
 		(fields_autoplaced yes)
 		(property "Reference" "R3"
-			(at 29.21 90.1699 0)
+			(at 41.91 90.1699 0)
 			(effects
 				(font
@@
 		)
 		(property "Value" "R_{T2}/100K"
-			(at 29.21 92.7099 0)
+			(at 41.91 92.7099 0)
 			(effects
 				(font
@@
 		)
 		(property "Footprint" ""
-			(at 24.892 91.44 90)
+			(at 37.592 91.44 90)
 			(effects
 				(font
@@
 		)
 		(property "Datasheet" "~"
-			(at 26.67 91.44 0)
+			(at 39.37 91.44 0)
 			(effects
 				(font
@@
 		)
 		(property "Description" "Resistor"
-			(at 26.67 91.44 0)
-			(effects
-				(font
+			(at 39.37 91.44 0)
+			(effects
+				(font
